Commit message: use proper nav2 servers

File: boat2023_nav2/src/description/boat2023.urdf (robot description, URDF)
Before this commit: robot boat2023, 1 links, 0 joints
Links:
- added link zed_depth_frame
- added link zed_link, mass 0.035; collision box size=0.015 0.130 0.022; visual box size=0.015 0.130 0.022
Joints:
- added joint zed_depth_joint: type fixed, parent zed_link, child zed_depth_frame, origin xyz=0 0 0 rpy=${-pi/2} 0 ${-pi/2}
- added joint zed_joint: type fixed, parent ego_vehicle, child zed_link, origin xyz=0.215 0 0.05 rpy=0 0 0

Commit message: fix gradient plugin linking

File: boat2023_nav2/src/description/boat2023.urdf (robot description, URDF)
Before this commit: robot boat2023, 3 links, 2 joints
Links:
- added link imu_link, mass 0.035; visual box size=0.1 0.1 0.1
Joints:
- added joint imu_joint: type fixed, parent ego_vehicle, child imu_link, origin xyz=0 0 0.01

Commit message: v0.1 costmap integration to nav2

File: boat2023_nav2/src/description/boat2023.urdf (robot description, URDF)
Before this commit: robot boat2023, 4 links, 3 joints
Links:
- removed link ego_vehicle
- removed link zed_depth_frame
- removed link zed_link
- added link base_link; collision box size=0.4 0.2 0.1; visual box size=1.14 0.735 0.475
- added link gps_link, mass 0.035; visual box size=0.1 0.1 0.1
Joints:
- removed joint zed_depth_joint
- removed joint zed_joint
- added joint gps_joint: type fixed, parent base_link, child gps_link, origin xyz=0 0 0.01
- joint imu_joint: parent ego_vehicle -> base_link

Commit message: add gnss link to ekf filter

File: boat2023_nav2/src/description/boat2023.urdf (robot description, URDF)
Before this commit: robot boat2023, 3 links, 2 joints
Links:
- removed link gps_link
- added link gnss_link, mass 0.035; visual box size=0.1 0.1 0.1
Joints:
- removed joint gps_joint
- added joint gnss_joint: type fixed, parent base_link, child gnss_link, origin xyz=0 0 0.01

Commit message: fix cams at comp

File: boat2023_nav2/src/description/boat2023.urdf (robot description, URDF)
Before this commit: robot boat2023, 3 links, 2 joints
Links:
- added link zed_link, mass 0.035; visual box size=0.1 0.1 0.1
Joints:
- added joint zed_joint: type fixed, parent base_link, child zed_link, origin xyz=0 0 0.01

Commit message: working comp BEV PCLs

File: boat2023_nav2/src/description/boat2023.urdf (robot description, URDF)
Before this commit: robot boat2023, 4 links, 3 joints
Links:
- removed link gnss_link
- removed link imu_link
- removed link zed_link
Joints:
- removed joint gnss_joint
- removed joint imu_joint
- removed joint zed_joint
